Commit message: seance 4

File: motoman_hc10_support/urdf/hc10.sensor.xacro (robot description, xacro)
@@ -4,5 +4,5 @@
     <xacro:macro name="hc10_sensor">
         <gazebo reference="camera_depth_frame">
-            <sensor name="kinect_camera" type="depth">
+            <sensor name="kinect" type="depth">
                 <update_rate>20</update_rate>
                 <camera>
@@ -28,5 +28,5 @@
                 <depthImageCameraInfoTopicName>/camera/depth/camera_info</depthImageCameraInfoTopicName>
                 <pointCloudTopicName>/camera/depth/points</pointCloudTopicName>
-                <frameName>camera_depth_frame</frameName>
+                <frameName>camera_depth_optical_frame</frameName>
                 <distortion_k1>0.0</distortion_k1>
                 <distortion_k2>0.0</distortion_k2>
@@ -41,5 +41,5 @@
         <link name="camera_depth_frame"/>
         <joint type="fixed" name="tool0_camera_joint">
-            <origin xyz="0 0 0" rpy="0 0 0"/>
+            <origin xyz="0 0 0" rpy="0 -1.5708 3.1415"/>
             <child link="camera_depth_frame"/>
             <parent link="tool0"/>
@@ -48,4 +48,13 @@
             <dynamics damping="1.0" friction="1.0"/>
         </joint>
+        <link name="camera_depth_optical_frame"/>
+        <joint type="fixed" name="camera_optical_joint">
+            <origin xyz="0 0 0" rpy="-1.5708 0 -1.5708"/>
+            <child link="camera_depth_optical_frame"/>
+            <parent link="camera_depth_frame"/>
+            <axis xyz="0 0 0" rpy="0 0 0"/>
+            <limit effort="10000" velocity="1000"/>
+            <dynamics damping="1.0" friction="1.0"/>
+        </joint>
     </xacro:macro>
 </robot>
